File: Electronics/SmallDSPDual/Analog_Input.kicad_sch (KiCad schematic)
At the start: 59 parts, among them J12 NC3FAAH2, J13 NC3FAAH2

Commit message: Generates Fabrication files for Maxi, Dual and In- nad Output Boards. Also Updates the ReadMe.
Parts:
- C? (x3): JLC Part Number C96446 -> (none); LCSC Part # (none) -> C96446
- C? (x5): JLC Part Number C307331 -> (none); LCSC Part # (none) -> C307331
- C? (x6): JLC Part Number C1848 -> (none); LCSC Part # (none) -> C1848
- C? (x4): JLC Part Number C1546 -> (none); LCSC Part # (none) -> C1546
- C? (x2): JLC Part Number C1555 -> (none); LCSC Part # (none) -> C1555
- D? (x4): JLC Part Number C78395 -> (none); LCSC Part # (none) -> C78395
- R? (x7): JLC Part Number C25076 -> (none); LCSC Part # (none) -> C25076
- R? (x4): JLC Part Number C25744 -> (none); LCSC Part # (none) -> C25744
- R? (x8): JLC Part Number C25741 -> (none); LCSC Part # (none) -> C25741
- R? (x4): JLC Part Number C25765 -> (none); LCSC Part # (none) -> C25765
- U? (x9): JLC Part Number C7426 -> (none); LCSC Part # (none) -> C7426
