File: Electronics/SmallDSPDual/Analog_Output.kicad_sch (KiCad schematic)
At the start: 77 parts, among them J14 NC3MAAH, J15 NC3MAAH

Commit message: Generates Fabrication files for Maxi, Dual and In- nad Output Boards. Also Updates the ReadMe.
Parts:
- C? (x4): JLC Part Number C1588 -> (none); LCSC Part # (none) -> C1588
- C? (x4): JLC Part Number C1555 -> (none); LCSC Part # (none) -> C1555
- C? (x2): JLC Part Number C1848 -> (none); LCSC Part # (none) -> C1848
- C? (x5): JLC Part Number C307331 -> (none); LCSC Part # (none) -> C307331
- C? (x2): JLC Part Number C96446 -> (none); LCSC Part # (none) -> C96446
- C? (x2): JLC Part Number C1546 -> (none); LCSC Part # (none) -> C1546
- C? (x4): JLC Part Number C13585 -> (none); LCSC Part # (none) -> C13585
- D? (x4): JLC Part Number C78395 -> (none); LCSC Part # (none) -> C78395
- R? (x4): JLC Part Number C25118 -> (none); LCSC Part # (none) -> C25118
- R? (x9): JLC Part Number C25744 -> (none); LCSC Part # (none) -> C25744
- R? (x4): JLC Part Number C11702 -> (none); LCSC Part # (none) -> C11702
- R? (x2): JLC Part Number C25905 -> (none); LCSC Part # (none) -> C25905
- R? (x2): JLC Part Number C25762 -> (none); LCSC Part # (none) -> C25762
- R? (x8): JLC Part Number C25765 -> (none); LCSC Part # (none) -> C25765
- R? (x2): JLC Part Number C25741 -> (none); LCSC Part # (none) -> C25741
- R? (x2): JLC Part Number C22980 -> (none); LCSC Part # (none) -> C22980
- U? (x12): JLC Part Number C7426 -> (none); LCSC Part # (none) -> C7426
