File: Electronics/SmallDSPDual/DSP_Decoupling.kicad_sch (KiCad schematic)
At the start: 25 parts

Commit message: Generates Fabrication files for Maxi, Dual and In- nad Output Boards. Also Updates the ReadMe.
Parts:
- C? (x11): JLC Part Number C307331 -> (none); LCSC Part # (none) -> C307331
- C? (x4): JLC Part Number C96446 -> (none); LCSC Part # (none) -> C96446
- C? (x4): JLC Part Number C52923 -> (none); LCSC Part # (none) -> C52923
- C? (x4): JLC Part Number C15195 -> (none); LCSC Part # (none) -> C15195
- R? (x2): JLC Part Number C25086 -> (none); LCSC Part # (none) -> C25086
