File: Electronics/SmallDSPDual/PSU.kicad_sch (KiCad schematic)
At the start: 39 parts, among them J16 Barrel_Jack_Switch, U13 LM317_TO-252, U14 LM317_TO-252, U15 LM317_TO-252

Commit message: Generates Fabrication files for Maxi, Dual and In- nad Output Boards. Also Updates the ReadMe.
Parts:
- C? (x7): JLC Part Number C28323 -> (none); LCSC Part # (none) -> C28323
- D? (x5): JLC Part Number C72041 -> (none); LCSC Part # (none) -> C72041
- FB? (x9): JLC Part Number C1017 -> (none); LCSC Part # (none) -> C1017
- Q? (x2): JLC Part Number C20526 -> (none); LCSC Part # (none) -> C20526
- R76, R79, R83: JLC Part Number C25862 -> (none); LCSC Part # (none) -> C25862
- R77: JLC Part Number C25924 -> (none); LCSC Part # (none) -> C25924
- R80: JLC Part Number C22980 -> (none); LCSC Part # (none) -> C22980
- R84, R?: JLC Part Number C22975 -> (none); LCSC Part # (none) -> C22975
- R86: JLC Part Number C23255 -> (none); LCSC Part # (none) -> C23255
- R?: JLC Part Number C22843 -> (none); LCSC Part # (none) -> C22843
- R?: JLC Part Number C23170 -> (none); LCSC Part # (none) -> C23170
- R?: JLC Part Number C23350 -> (none); LCSC Part # (none) -> C23350
- U13, U14, U15: JLC Part Number C75510 -> (none); LCSC Part # (none) -> C75510
