File: Electronics/SmallDSPDual/SmallDSPDual.kicad_sch (KiCad schematic)
At the start: 68 parts, among them J1 Header, J10 Header, J11 Programming, J2 Header, J3 Header, J4 Header, J5 Header, J6 Header, J7 Header, J8 Header, J9 Header, Q1 NSS1C300ET4G, SW1 TS-1187A-B-A-B, SW2 CJS-1201TB, U1 ADAU1463, U2 ADM811, U3 M95M01-R, Y1 830105957509

Commit message: Generates Fabrication files for Maxi, Dual and In- nad Output Boards. Also Updates the ReadMe.
Parts:
- C1, C2, C7: JLC Part Number C307331 -> (none); LCSC Part # (none) -> C307331
- C3: JLC Part Number C1527 -> (none); LCSC Part # (none) -> C1527
- C5, C6: JLC Part Number C1557 -> (none); LCSC Part # (none) -> C1557
- C8: JLC Part Number C96446 -> (none); LCSC Part # (none) -> C96446
- D1, D2, D3, D4, D5, D6: JLC Part Number C78395 -> (none); LCSC Part # (none) -> C78395
- D7: JLC Part Number C72041 -> (none); LCSC Part # (none) -> C72041
- R1, R10, R11, R12, R17, R2, R3, R4, R5, R6, R7, R8, R9: JLC Part Number C25076 -> (none); LCSC Part # (none) -> C25076
- R13: JLC Part Number C25741 -> (none); LCSC Part # (none) -> C25741
- R14, R16, R19: JLC Part Number C11702 -> (none); LCSC Part # (none) -> C11702
- R15: JLC Part Number C25744 -> (none); LCSC Part # (none) -> C25744
- R18: JLC Part Number C23159 -> (none); LCSC Part # (none) -> C23159
- SW1: JLC Part Number C318884 -> (none); LCSC Part # (none) -> C318884
Other:
- title: SmallDSP -> SmallDSP Dual
